File: HARDWARE/ETH1IRCAM1/ETH1IRCAM1.kicad_sch (KiCad schematic)
At the start: 4 parts

Commit message: PCB changes
Parts:
- added H105, H106, H107, H108: M3, MountingHole:MountingHole_3.2mm_M3_DIN965_Pad_TopBottom, symbol Mechanical:MountingHole
Changed lines of the file:
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@@
     (stroke (width 0) (type default))
+  )
+  (symbol (lib_id "Mechanical:MountingHole") (at 95.885 190.5 0) (unit 1)
+    (in_bom yes) (on_board yes) (dnp no) (fields_autoplaced)
+    (property "Reference" "H107" (at 98.425 189.23 0)
+      (effects (font (size 1.27 1.27)) (justify left))
+    )
+    (property "Value" "M3" (at 98.425 191.77 0)
+      (effects (font (size 1.27 1.27)) (justify left))
+    )
+    (property "Footprint" "MountingHole:MountingHole_3.2mm_M3_DIN965_Pad_TopBottom" (at 95.885 190.5 0)
+      (effects (font (size 1.27 1.27)) hide)
+    )
+    (property "Datasheet" "~" (at 95.885 190.5 0)
+      (effects (font (size 1.27 1.27)) hide)
+    )
+    (instances
+      (project "ETH1IRCAM1"
+        (path "/f8ed47a9-95cb-42d4-bd7f-c1b2ff57d6fd"
+          (reference "H107") (unit 1)
+        )
+      )
+    )
   )
   (symbol (lib_id "Mechanical:MountingHole") (at 19.05 190.5 0) (unit 1)
@@
     )
   )
+  (symbol (lib_id "Mechanical:MountingHole") (at 70.485 190.5 0) (unit 1)
+    (in_bom yes) (on_board yes) (dnp no) (fields_autoplaced)
+    (property "Reference" "H105" (at 73.025 189.23 0)
+      (effects (font (size 1.27 1.27)) (justify left))
+    )
+    (property "Value" "M3" (at 73.025 191.77 0)
+      (effects (font (size 1.27 1.27)) (justify left))
+    )
+    (property "Footprint" "MountingHole:MountingHole_3.2mm_M3_DIN965_Pad_TopBottom" (at 70.485 190.5 0)
+      (effects (font (size 1.27 1.27)) hide)
+    )
+    (property "Datasheet" "~" (at 70.485 190.5 0)
+      (effects (font (size 1.27 1.27)) hide)
+    )
+    (instances
+      (project "ETH1IRCAM1"
+        (path "/f8ed47a9-95cb-42d4-bd7f-c1b2ff57d6fd"
+          (reference "H105") (unit 1)
+        )
+      )
+    )
+  )
   (symbol (lib_id "Mechanical:MountingHole") (at 31.75 190.5 0) (unit 1)
     (in_bom yes) (on_board yes) (dnp no) (fields_autoplaced)
@@
         (path "/f8ed47a9-95cb-42d4-bd7f-c1b2ff57d6fd"
           (reference "H102") (unit 1)
+        )
+      )
+    )
+  )
+  (symbol (lib_id "Mechanical:MountingHole") (at 108.585 190.5 0) (unit 1)
+    (in_bom yes) (on_board yes) (dnp no) (fields_autoplaced)
+    (property "Reference" "H108" (at 111.125 189.23 0)
+      (effects (font (size 1.27 1.27)) (justify left))
+    )
+    (property "Value" "M3" (at 111.125 191.77 0)
+      (effects (font (size 1.27 1.27)) (justify left))
+    )
+    (property "Footprint" "MountingHole:MountingHole_3.2mm_M3_DIN965_Pad_TopBottom" (at 108.585 190.5 0)
+      (effects (font (size 1.27 1.27)) hide)
+    )
+    (property "Datasheet" "~" (at 108.585 190.5 0)
+      (effects (font (size 1.27 1.27)) hide)
+    )
+    (instances
+      (project "ETH1IRCAM1"
+        (path "/f8ed47a9-95cb-42d4-bd7f-c1b2ff57d6fd"
+          (reference "H108") (unit 1)
         )
       )
@@
         )
       )
+    )
+  )
+  (symbol (lib_id "Mechanical:MountingHole") (at 83.185 190.5 0) (unit 1)
+    (in_bom yes) (on_board yes) (dnp no) (fields_autoplaced)
+    (property "Reference" "H106" (at 85.725 189.23 0)
+      (effects (font (size 1.27 1.27)) (justify left))
+    )
+    (property "Value" "M3" (at 85.725 191.77 0)
+      (effects (font (size 1.27 1.27)) (justify left))
+    )
+    (property "Footprint" "MountingHole:MountingHole_3.2mm_M3_DIN965_Pad_TopBottom" (at 83.185 190.5 0)
+      (effects (font (size 1.27 1.27)) hide)
+    )
+    (property "Datasheet" "~" (at 83.185 190.5 0)
+      (effects (font (size 1.27 1.27)) hide)
+    )
+    (instances
+      (project "ETH1IRCAM1"
+        (path "/f8ed47a9-95cb-42d4-bd7f-c1b2ff57d6fd"
+          (reference "H106") (unit 1)
+        )
+      )
