File: HARDWARE/ETH1IRCAM1/ETH1IRCAM1.kicad_sch (KiCad schematic)
At the start: 8 parts

Commit message: PCB changes
Parts:
- added FID101, FID102, FID103, FID104: Fiducial, Fiducial:Fiducial_1.5mm_Mask3mm, symbol Mechanical:Fiducial
- added HS101: 960-19-12-S-AB-0, ETH1IRCAM1:960-19-12-S-AB-0, symbol Mechanical:Heatsink
- H101, H102, H103, H104, H105, H106, H107, H108: now left out of the parts list
Other:
- note added: "TG-A2200-10-10-1.5"
