File: HARDWARE/ETH1IRCAM1/ETH1IRCAM1.kicad_pcb (KiCad board)
At the start: 4 copper layers, 75 x 45 mm, 107 parts, among them J201 MKDS 1,5/ 2-5,08, J301 RJ45_Wuerth_7499010121A, J401 20021111-00010T4LF, Q201 SI5618A, Q202 MMBT3904, Q501 MMBT3904, U201 TSR_1-2450, U202 TLV62568DBV, U203 TLV75530PDBV, U204 MIC5365-2.8YD5, U205 MIC5365-1.2YD5, U301 LAN8742A, U401 STM32H723VETx, U402 24LC08B-E/MS, U501 105028-1001 + Lepton 3.1R, X501 ASEMB-25.000MHZ-LY-T, Y301 NX5032GA-25, Y401 NX5032GA-16

Commit message: PCB changes
Parts:
- added H105: M3, MountingHole:MountingHole_3.2mm_M3_DIN965_Pad_TopBottom, F.Cu at (129.0, 81.0)
- added H106: M3, MountingHole:MountingHole_3.2mm_M3_DIN965_Pad_TopBottom, F.Cu at (150.0, 119.0)
- added H107: M3, MountingHole:MountingHole_3.2mm_M3_DIN965_Pad_TopBottom, F.Cu at (150.0, 81.0)
- added H108: M3, MountingHole:MountingHole_3.2mm_M3_DIN965_Pad_TopBottom, F.Cu at (129.0, 119.0)
- moved JP401 8.83 mm to (140.2, 82.0), turned to 0 degrees
- moved H101 5.00 mm to (113.0, 81.0)
- moved H104 5.00 mm to (113.0, 119.0)
Routing:
- net /MCU/MCU_DEFAULT: track 5.50 -> 12.8 mm
Other:
- board size 75 x 45 mm -> 80 x 45 mm
- board text added: "ETH1IRCAM1 V1.2 DEFAULT IP: 192.168.1.56"
- board text added: "SHORT JP401 FOR DEF. CFG"
- board text removed: "ETH1IRCAM1 V1.1 DEFAULT IP: 192.168.1.56"
- board text removed: "SHORT JP401 FOR DEFAULT CONFIGURATION"

Commit message: PCB changes
Parts:
- Q501, R503, R506: moved to B.Cu
- moved C205 4.06 mm to (121.3, 87.5)
- moved C206 4.06 mm to (117.1, 87.5)
- moved C208 4.06 mm to (125.0, 88.8)
- moved C209 4.06 mm to (117.1, 89.8)
- moved U203 4.06 mm to (121.3, 88.6)
- moved U204 4.06 mm to (117.1, 88.6)
- moved R506 2.29 mm to (129.7, 92.5), turned to 0 degrees
- moved C207 1.73 mm to (124.0, 111.9)
- moved C210 1.73 mm to (124.0, 109.6)
- moved U205 1.73 mm to (124.0, 110.7)
- moved C505 0.13 mm to (129.7, 94.9)
- moved R503 0.13 mm to (129.7, 101.5)
- turned Q501 to 0 degrees
Routing:
- net /Lepton/LEP_~{RST}: track 3.57 -> 6.96 mm, vias 0 -> 1
- net /Lepton/LEP_nRST: track 21.1 -> 24.4 mm
- net +2V8: track 3.98 -> 5.68 mm, vias 2 -> 3
- net Net-(Q501-B): track 3.83 -> 2.36 mm
- net +1V2: track 3.56 -> 4.88 mm, vias 2 -> 3
Other:
- board text added: "ETH1IRCAM1 V1.3 DEFAULT IP: 192.168.1.56"
- board text removed: "ETH1IRCAM1 V1.2 DEFAULT IP: 192.168.1.56"
