File: HARDWARE/ETH1IRCAM1/ETH1IRCAM1.kicad_pcb (KiCad board)
At the start: 4 copper layers, 80 x 45 mm, 111 parts, among them J201 MKDS 1,5/ 2-5,08, J301 RJ45_Wuerth_7499010121A, J401 20021111-00010T4LF, Q201 SI5618A, Q202 MMBT3904, Q501 MMBT3904, U201 TSR_1-2450, U202 TLV62568DBV, U203 TLV75530PDBV, U204 MIC5365-2.8YD5, U205 MIC5365-1.2YD5, U301 LAN8742A, U401 STM32H723VETx, U402 24LC08B-E/MS, U501 105028-1001 + Lepton 3.1R, X501 ASEMB-25.000MHZ-LY-T, Y301 NX5032GA-25, Y401 NX5032GA-16

Commit message: PCB changes
Parts:
- removed R307, R308, R309, R311: 10k, Resistor_SMD:R_0603_1608Metric_Pad0.98x0.95mm_HandSolder
- removed R310: 1k5, Resistor_SMD:R_0603_1608Metric_Pad0.98x0.95mm_HandSolder
- removed R312: 12k1, Resistor_SMD:R_0603_1608Metric_Pad0.98x0.95mm_HandSolder
- removed R313, R314, R315, R316: 49R9, Resistor_SMD:R_0603_1608Metric_Pad0.98x0.95mm_HandSolder
- removed R317, R318: 560, Resistor_SMD:R_0603_1608Metric_Pad0.98x0.95mm_HandSolder
- added FID101: Fiducial, Fiducial:Fiducial_1.5mm_Mask3mm, F.Cu at (99.9, 81.0)
- added FID102: Fiducial, Fiducial:Fiducial_1.5mm_Mask3mm, B.Cu at (99.9, 81.0)
- added FID103: Fiducial, Fiducial:Fiducial_1.5mm_Mask3mm, F.Cu at (178.9, 120.1)
- added FID104: Fiducial, Fiducial:Fiducial_1.5mm_Mask3mm, B.Cu at (178.9, 120.1)
- added HS101: 960-19-12-S-AB-0, ETH1IRCAM1:960-19-12-S-AB-0, F.Cu at (140.1, 98.0)
- added RN301: EXB-V8V330JV, Resistor_SMD:R_Array_Concave_4x0603, F.Cu at (153.2, 94.1)
- added RN302: EXB-V8V103JV, Resistor_SMD:R_Array_Concave_4x0603, B.Cu at (153.2, 94.1)
- added RN303: EXB-38V510JV, Resistor_SMD:R_Array_Concave_4x0603, B.Cu at (175.4, 92.7)
- C302, C305, C306, R303, R404, R405, U402: moved to B.Cu
- C303, C409, R401: moved to F.Cu
- R301: value 33 -> 10k
- R302: value 33 -> 1k5; moved to B.Cu
- R304: value 33 -> 12k1; moved to B.Cu
- R305: value 33 -> 560; moved to B.Cu
- R306: value 10k -> 560
- moved H105 37.9 mm to (93.0, 93.0)
- moved H108 37.9 mm to (93.0, 107.0)
- moved H106 26.5 mm to (123.5, 119.0)
- moved H107 26.5 mm to (123.5, 81.0)
- moved H101 20.0 mm to (93.0, 81.0)
- moved H104 20.0 mm to (93.0, 119.0)
- moved U402 16.1 mm to (139.4, 97.2), turned to 0 degrees
- moved C414 14.7 mm to (139.4, 99.9), turned to 0 degrees
- moved R306 14.0 mm to (166.4, 86.9), turned to 90 degrees
- moved C312 13.6 mm to (169.9, 100.3), turned to -90 degrees
- moved R303 13.2 mm to (166.4, 100.3), turned to -90 degrees
- moved R305 12.6 mm to (166.4, 96.8), turned to -90 degrees
- moved C207 12.3 mm to (112.0, 114.7)
- moved C210 12.3 mm to (112.0, 112.5)
- moved U205 12.2 mm to (112.0, 113.6)
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Connections:
- R301 pad 1: /Ethernet/MODE0 -> GND
- R301 pad 2: /Ethernet/RMII_RXD0 -> Net-(U301-RXER/PHYAD0)
- R302 pad 1: /Ethernet/MODE1 -> +3.3V
- R302 pad 2: /Ethernet/RMII_RXD1 -> /Ethernet/RMII_MDIO
- R303 pad 1: Net-(U301-RXER/PHYAD0) -> /Ethernet/LED2
- R304 pad 1: /Ethernet/MODE2 -> GND
- R304 pad 2: /Ethernet/RMII_CRS_DV -> Net-(U301-RBIAS)
- R305 pad 1: /Ethernet/REFCLK0 -> Net-(J301-Pad11)
- R305 pad 2: /Ethernet/REF_CLK -> GND
- R306 pad 1: +3.3V -> Net-(J301-Pad9)
- R306 pad 2: /Ethernet/MODE0 -> GND
Routing:
- net +3.3V: track 44.5 -> 84.2 mm, vias 20 -> 22
- net VCCQ: track 58.0 -> 38.5 mm, vias 4 -> 3
- net /MCU/TCK_SWCLK: track 6.89 -> 23.5 mm, vias 0 -> 1
- net /MCU/TMS_SWDIO: track 6.86 -> 23.2 mm, vias 0 -> 1
- net /Lepton/SPI_MISO: track 15.5 -> 31.4 mm
- net /Lepton/I2C4_SCL: track 29.1 -> 44.6 mm
- net GND: track 50.4 -> 65.4 mm, vias 18 -> 29
- net /Lepton/SPI_CLK: track 15.2 -> 28.7 mm
- net /Lepton/LEP_~{RST}: track 6.96 -> 18.0 mm
- net /MCU/I2C1_SCL: track 18.1 -> 7.26 mm, vias 2 -> 1
- net /Lepton/I2C4_SDA: track 31.1 -> 41.8 mm
- net /Lepton/SPI_~{SS}: track 15.5 -> 26.1 mm
- net /MCU/I2C1_SDA: track 17.5 -> 7.03 mm, vias 2 -> 1
- net /MCU/EEPROM_WP: track 16.3 -> 6.64 mm, vias 2 -> 1
- net /MCU/NRST: track 52.5 -> 58.7 mm, vias 1 -> 3
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Other:
- board size 80 x 45 mm -> 100 x 45 mm
- board text added: "ETH1IRCAM1 V1.4 DEFAULT IP: 192.168.1.56"
- board text removed: "ETH1IRCAM1 V1.3 DEFAULT IP: 192.168.1.56"
