File: HARDWARE/ETH1IRCAM1/MCU.kicad_sch (KiCad schematic)
At the start: 27 parts, among them J401 20021111-00010T4LF, U401 STM32H723VETx, U402 24LC08B-E/MS, Y401 NX5032GA-16

Commit message: Bug fixes
Other:
- moved on the sheet: C401, C402, C403, C404, C405, C407, C408, C409, C410, C411, C412, C413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
