File: HARDWARE/ETH1IRCAM1/Power.kicad_sch (KiCad schematic)
At the start: 28 parts, among them J201 MKDS 1,5/ 2-5,08, Q201 SI5618A, Q202 MMBT3904, U201 TSR_1-2450, U202 TLV62568DBV, U203 TLV75530PDBV, U204 MIC5365-2.8YD5, U205 MIC5365-1.2YD5

Commit message: Bug fixes
Other:
- moved on the sheet: C201, C202, C203, C205, C206, C208, C209, C210, D201, D202, L201, Q201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
